Commit message: Added Docker, Made the entire robot and fixed mapping

File: nolon_bot_description/urdf/mobile_base/mobile_base.control.xacro (robot description, xacro)
@@ -64,9 +64,3 @@
         </joint>
     </ros2_control>
-    <gazebo>
-        <plugin filename="libgz_ros2_control-system.so" name="gz_ros2_control::GazeboSimROS2ControlPlugin">
-            <parameters>$(find nolon_bot_description)/config/nolon_bot_control.yaml</parameters>
-            <controller_manager_node_name>controller_manager</controller_manager_node_name>
-        </plugin>
-    </gazebo>
 </robot>

File: nolon_bot_description/urdf/nolon_bot.urdf.xacro (robot description, xacro)
@@ -16,11 +16,35 @@
 -->
 <robot xmlns:xacro="http://www.ros.org/wiki/xacro" name="nolon_bot">
+    <xacro:property name="use_lidar" value="false"/>
     <xacro:include filename="mobile_base/mobile_base.urdf.xacro"/>
     <xacro:include filename="mobile_base/mobile_base.control.xacro"/>
-    <xacro:include filename="sensors/lidar.sensor.xacro"/>
-    <joint name="lidar_joint" type="fixed">
+    <xacro:include filename="containment/containment_box.urdf.xacro"/>
+    <xacro:include filename="robotic_arm/robotic_arm.urdf.xacro"/>
+    <xacro:include filename="robotic_arm/robotic_arm.control.xacro"/>
+    <xacro:if value="${use_lidar}">
+        <xacro:include filename="sensors/lidar.sensor.xacro"/>
+        <joint name="lidar_joint" type="fixed">
+            <parent link="base_link"/>
+            <child link="lidar_link"/>
+            <origin xyz="0 0 0" rpy="0 0 0"/>
+        </joint>
+    </xacro:if>
+<!-- -0.1 0 0.5-->
+    <joint name="containment_to_mobile_base" type="fixed">
         <parent link="base_link"/>
-        <child link="lidar_link"/>
-        <origin xyz="-0.1 0 0.5" rpy="0 0 0"/>
+        <child link="containment_box"/>
+        <origin xyz="0 0 0" rpy="0 0 0"/>
     </joint>
+    <!-- <link name="world"/> -->
+    <joint name="robotic_arm_to_containment" type="fixed">
+        <parent link="containment_box"/>
+        <child link="link_base"/>
+        <origin xyz="-0.25 0.1 0.8" rpy="0 0 3.14159"/>
+    </joint>
+    <gazebo>
+        <plugin filename="libgz_ros2_control-system.so" name="gz_ros2_control::GazeboSimROS2ControlPlugin">
+            <parameters>$(find nolon_bot_description)/config/nolon_bot_control.yaml</parameters>
+            <controller_manager_node_name>controller_manager</controller_manager_node_name>
+        </plugin>
+    </gazebo>
 </robot>

File: nolon_bot_description/urdf/robotic_arm/robotic_arm.urdf.xacro (robot description, xacro)
@@ -1,22 +1,21 @@
 <?xml version="1.0"?>
 <!--
-nolon_bot Robotic Arm URDF
+XArm 6-DOF Robotic Arm URDF (Converted Format)
 Author: Aayush Rath | Date: 10/08/2025
-Defines the URDF model for a 6-DOF robotic arm using STL meshes.
+Defines the URDF model for a 6-DOF XArm robotic arm using STL/OBJ meshes.
 Implements Xacro macros for reusable link and joint definitions,
 with conditional mesh path resolution for Gazebo or RViz usage.
 Includes:
 - `mesh_link` macro for defining links with visual, collision, and inertial properties
-- `fixed_joint` macro for rigidly connecting links
+- `revolute_joint` macro for defining revolute joints with limits
 - Conditional `mesh_path` property based on `use_gazebo` argument
-- Base link, arm segments, and transient connection meshes
+- Base link and 6 arm links with proper kinematic chain
 Usage:
 - Set `use_gazebo` argument to `true` for simulation with Gazebo, or `false` for RViz-only usage
-- Place STL meshes in the `meshes/robotic_arm/` directory
+- Place STL/OBJ meshes in the `meshes/robotic_arm/` directory
 - Launch with:
   `ros2 launch urdf_tutorial display.launch.py model:=<path_to_this_file> use_gazebo:=true`
-- Modify joint types for actuation as needed
 -->
-<robot xmlns:xacro="http://www.ros.org/wiki/xacro" name="robot_name">
+<robot xmlns:xacro="http://www.ros.org/wiki/xacro" name="robotic_arm">
     <!-- ================= CHECK USAGE ================= -->
     <xacro:arg name="use_gazebo" default="true"/>
@@ -26,20 +25,28 @@
     </xacro:if>
     <xacro:unless value="$(arg use_gazebo)">
-        <xacro:property name="mesh_path" value="$(find nolon_bot_description)/meshes/"/>
+        <xacro:property name="mesh_path" value="$(find nolon_bot_description)/meshes/robotic_arm/"/>
     </xacro:unless>
+    <!-- ================= MATERIALS ================= -->
+    <material name="White">
+        <color rgba="1.0 1.0 1.0 1.0"/>
+    </material>
+    <material name="Silver">
+        <color rgba="0.75 0.75 0.75 1.0"/>
+    </material>
     <!-- ================= MACROS ================= -->
-    <!-- Generic mesh link -->
-    <xacro:macro name="mesh_link" params="name mesh mass ixx iyy izz ixy ixz iyz ox oy oz orx ory orz">
+    <!-- Generic mesh link with separate visual and collision meshes -->
+    <xacro:macro name="mesh_link" params="name visual_mesh collision_mesh mass ixx iyy izz ixy ixz iyz ox oy oz orx ory orz material_name:=White">
         <link name="${name}">
             <visual>
                 <origin xyz="${ox} ${oy} ${oz}" rpy="${orx} ${ory} ${orz}"/>
                 <geometry>
-                    <mesh filename="${mesh_path}${mesh}"/>
+                    <mesh filename="${mesh_path}${visual_mesh}.stl"/>
                 </geometry>
+                <material name="${material_name}"/>
             </visual>
             <collision>
                 <origin xyz="${ox} ${oy} ${oz}" rpy="${orx} ${ory} ${orz}"/>
                 <geometry>
-                    <mesh filename="${mesh_path}${mesh}"/>
+                    <mesh filename="${mesh_path}${collision_mesh}.stl"/>
                 </geometry>
             </collision>
@@ -51,15 +58,7 @@
         </link>
     </xacro:macro>
-    <!-- Fixed joint -->
-    <xacro:macro name="fixed_joint" params="parent child ox oy oz orx ory orz">
-        <joint name="${parent}_to_${child}" type="fixed">
-            <parent link="${parent}"/>
-            <child link="${child}"/>
-            <origin xyz="${ox} ${oy} ${oz}" rpy="${orx} ${ory} ${orz}"/>
-        </joint>
-    </xacro:macro>
     <!-- Revolute joint -->
-    <xacro:macro name="revolute_joint" params="parent child ax ay az ox oy oz orx ory orz lower upper effort vel">
-        <joint name="${parent}_to_${child}" type="revolute">
+    <xacro:macro name="revolute_joint" params="name parent child ax ay az ox oy oz orx ory orz lower upper effort vel">
+        <joint name="${name}" type="revolute">
             <parent link="${parent}"/>
             <child link="${child}"/>
@@ -67,35 +66,67 @@
             <origin xyz="${ox} ${oy} ${oz}" rpy="${orx} ${ory} ${orz}"/>
             <limit lower="${lower}" upper="${upper}" effort="${effort}" velocity="${vel}"/>
+            <dynamics damping="1.0" friction="1.0"/>
         </joint>
     </xacro:macro>
     <!-- ================= ROBOT STRUCTURE ================= -->
-    <!-- BASE LINKS -->
-    <link name="base_link"/>
-    <xacro:mesh_link name="link1" mesh="link1.stl" mass="1.0" ixx="1.0" iyy="1.0" izz="1.0" ixy="0" ixz="0" iyz="0" ox="0.2580" oy="-0.0652" oz="-0.7945" orx="0" ory="0" orz="0"/>
-    <xacro:fixed_joint parent="base_link" child="link1" ox="-0.2580" oy="0.0652" oz="0.7945" orx="0" ory="0" orz="0"/>
+    <!-- BASE LINK -->
+    <link name="link_base">
+        <visual>
+            <origin xyz="0 0 0" rpy="0 0 0"/>
+            <geometry>
+                <mesh filename="${mesh_path}link_base.stl"/>
+            </geometry>
+            <material name="White"/>
+        </visual>
+        <collision>
+            <origin xyz="0 0 0" rpy="0 0 0"/>
+            <geometry>
+                <mesh filename="${mesh_path}link_base.stl"/>
+            </geometry>
+        </collision>
+        <inertial>
+            <origin xyz="0.0 0.0 0.09103" rpy="0 0 0"/>
+            <mass value="0.01"/>
+            <inertia ixx="0.00494875" ixy="-3.5E-06" ixz="1.25E-05"
+                     iyy="0.00494174" iyz="1.67E-06" izz="0.002219"/>
+        </inertial>
+    </link>
     <!-- ARM LINKS -->
-    <xacro:mesh_link name="link2" mesh="link2.stl" mass="1.0" ixx="1.0" iyy="1.0" izz="1.0" ixy="0" ixz="0" iyz="0" ox="0.2580" oy="-0.0652" oz="-0.9739" orx="0" ory="0" orz="0"/>
-    <xacro:mesh_link name="link3" mesh="link3.stl" mass="1.0" ixx="1.0" iyy="1.0" izz="1.0" ixy="0" ixz="0" iyz="0" ox="0.2572" oy="-0.1421" oz="-1.1105" orx="0" ory="0" orz="0"/>
-    <xacro:mesh_link name="link4" mesh="link4.stl" mass="1.0" ixx="1.0" iyy="1.0" izz="1.0" ixy="0" ixz="0" iyz="0" ox="0.0755" oy="-0.1198" oz="-1.4001" orx="0" ory="0" orz="0"/>
-    <xacro:mesh_link name="link5" mesh="link5.stl" mass="1.0" ixx="1.0" iyy="1.0" izz="1.0" ixy="0" ixz="0" iyz="0" ox="-0.1375" oy="-0.0633" oz="-1.4383" orx="0" ory="0" orz="0"/>
-    <xacro:mesh_link name="link6" mesh="link6.stl" mass="1.0" ixx="1.0" iyy="1.0" izz="1.0" ixy="0" ixz="0" iyz="0" ox="0" oy="0" oz="0" orx="0" ory="0" orz="0"/>
-    <!-- ARM TRANSIENTS -->
-    <xacro:mesh_link name="link1-2" mesh="link1-2.stl" mass="1.0" ixx="1.0" iyy="1.0" izz="1.0" ixy="0" ixz="0" iyz="0" ox="0.2580" oy="-0.0652" oz="-0.9325" orx="0" ory="0" orz="0"/>
-    <xacro:mesh_link name="link2-3" mesh="link2-3.stl" mass="1.0" ixx="1.0" iyy="1.0" izz="1.0" ixy="0" ixz="0" iyz="0" ox="0.2572" oy="-0.1020" oz="-1.1105" orx="0" ory="0" orz="0"/>
-    <xacro:mesh_link name="link3-4" mesh="link3-4.stl" mass="1.0" ixx="1.0" iyy="1.0" izz="1.0" ixy="0" ixz="0" iyz="0" ox="0.0755" oy="-0.0830" oz="-1.4001" orx="0" ory="0" orz="0"/>
-    <xacro:mesh_link name="link4-5" mesh="link4-5.stl" mass="1.0" ixx="1.0" iyy="1.0" izz="1.0" ixy="0" ixz="0" iyz="0" ox="-0.0994" oy="-0.0635" oz="-1.4448" orx="0" ory="0" orz="0"/>
-    <xacro:mesh_link name="link5-6" mesh="link5-6.stl" mass="1.0" ixx="1.0" iyy="1.0" izz="1.0" ixy="0" ixz="0" iyz="0" ox="0" oy="0" oz="0" orx="0" ory="0" orz="0"/>
-    <xacro:mesh_link name="link6-ee" mesh="link6-ee.stl" mass="1.0" ixx="1.0" iyy="1.0" izz="1.0" ixy="0" ixz="0" iyz="0" ox="0" oy="0" oz="0" orx="0" ory="0" orz="0"/>
-    <!-- ARM JOINTS (Fixed for now) -->
-    <xacro:fixed_joint parent="link1" child="link1-2" ox="${-0.2580+0.2580}" oy="${0.0652-0.0652}" oz="${0.9325-0.7945}" orx="0" ory="0" orz="0"/>
-    <xacro:revolute_joint parent="link1-2" child="link2" ox="${-0.2580+0.2580}" oy="${0.0652-0.0652}" oz="${0.9739-0.9325}" orx="0" ory="0" orz="0" ax="0" ay="0" az="1" lower="0" upper="5" effort="0" vel="0"/>
-    <xacro:fixed_joint parent="link2" child="link2-3" ox="${-0.2572+0.2580}" oy="${0.1020-0.0652}" oz="${1.1105-0.9739}" orx="0" ory="0" orz="0"/>
-    <xacro:revolute_joint parent="link2-3" child="link3" ox="${-0.2572+0.2572}" oy="${0.1421-0.1020}" oz="${1.1105-1.1105}" orx="0" ory="0" orz="0" ax="0" ay="1" az="0" lower="0" upper="5" effort="0" vel="0"/>
-    <xacro:fixed_joint parent="link3" child="link3-4" ox="${-0.0755+0.2572}" oy="${0.0830-0.1421}" oz="${1.4001-1.1105}" orx="0" ory="0" orz="0"/>
-    <xacro:revolute_joint parent="link3-4" child="link4" ox="${-0.0755+0.0755}" oy="${0.1198-0.0830}" oz="${1.4001-1.4001}" orx="0" ory="0" orz="0" ax="0" ay="1" az="0" lower="0" upper="5" effort="0" vel="0"/>
-    <xacro:fixed_joint parent="link4" child="link4-5" ox="${0.0994+0.0755}" oy="${0.0635-0.1198}" oz="${1.4448-1.4001}" orx="0" ory="0.09" orz="0"/>
-    <xacro:revolute_joint parent="link4-5" child="link5" ox="${0.1375-0.0994}" oy="${0.0633-0.0635}" oz="${1.4383-1.4448}" orx="0" ory="0" orz="0" ax="0.9736" ay="0" az="-0.2279" lower="0" upper="${2*pi}" effort="0" vel="0"/>
-    <xacro:fixed_joint parent="link5" child="link5-6" ox="0" oy="0" oz="0" orx="0" ory="0" orz="0"/>
-    <xacro:fixed_joint parent="link5-6" child="link6" ox="0" oy="0" oz="0" orx="0" ory="0" orz="0"/>
-    <xacro:fixed_joint parent="link6" child="link6-ee" ox="0" oy="0" oz="0" orx="0" ory="0" orz="0"/>
+    <xacro:mesh_link name="link1" visual_mesh="link1" collision_mesh="link1"
+                     mass="0.01" ixx="0.001" iyy="0.001" izz="0.001" ixy="0" ixz="0" iyz="0"
+                     ox="0" oy="0" oz="0" orx="0" ory="0" orz="0" material_name="White"/>
+    <xacro:mesh_link name="link2" visual_mesh="link2" collision_mesh="link2"
+                     mass="0.01" ixx="0.001" iyy="0.001" izz="0.001" ixy="0" ixz="0" iyz="0"
+                     ox="0" oy="0" oz="0" orx="0" ory="0" orz="0" material_name="White"/>
+    <xacro:mesh_link name="link3" visual_mesh="link3" collision_mesh="link3"
+                     mass="0.01" ixx="0.001" iyy="0.001" izz="0.001" ixy="0" ixz="0" iyz="0"
+                     ox="0" oy="0" oz="0" orx="0" ory="0" orz="0" material_name="White"/>
+    <xacro:mesh_link name="link4" visual_mesh="link4" collision_mesh="link4"
+                     mass="0.01" ixx="0.001" iyy="0.001" izz="0.001" ixy="0" ixz="0" iyz="0"
+                     ox="0" oy="0" oz="0" orx="0" ory="0" orz="0" material_name="White"/>
+    <xacro:mesh_link name="link5" visual_mesh="link5" collision_mesh="link5"
+                     mass="0.01" ixx="0.001" iyy="0.001" izz="0.001" ixy="0" ixz="0" iyz="0"
+                     ox="0" oy="0" oz="0" orx="0" ory="0" orz="0" material_name="White"/>
+    <xacro:mesh_link name="link6" visual_mesh="link6" collision_mesh="link6"
+                     mass="0.01" ixx="0.001" iyy="0.001" izz="0.001" ixy="0" ixz="0" iyz="0"
+                     ox="0" oy="0" oz="0" orx="0" ory="0" orz="0" material_name="Silver"/>
+    <!-- ARM JOINTS -->
+    <xacro:revolute_joint name="joint1" parent="link_base" child="link1"
+                          ax="0" ay="0" az="1" ox="0" oy="0" oz="0.267" orx="0" ory="0" orz="0"
+                          lower="-${2*pi}" upper="${2*pi}" effort="50.0" vel="3.14"/>
+    <xacro:revolute_joint name="joint2" parent="link1" child="link2"
+                          ax="0" ay="0" az="1" ox="0" oy="0" oz="0" orx="-1.5708" ory="0" orz="0"
+                          lower="-2.059" upper="2.0944" effort="50.0" vel="3.14"/>
+    <xacro:revolute_joint name="joint3" parent="link2" child="link3"
+                          ax="0" ay="0" az="1" ox="0.0535" oy="-0.2845" oz="0" orx="0" ory="0" orz="0"
+                          lower="-3.927" upper="0.19198" effort="32.0" vel="3.14"/>
+    <xacro:revolute_joint name="joint4" parent="link3" child="link4"
+                          ax="0" ay="0" az="1" ox="0.0775" oy="0.3425" oz="0" orx="-1.5708" ory="0" orz="0"
+                          lower="-${2*pi}" upper="${2*pi}" effort="32.0" vel="3.14"/>
+    <xacro:revolute_joint name="joint5" parent="link4" child="link5"
+                          ax="0" ay="0" az="1" ox="0" oy="0" oz="0" orx="0" ory="0" orz="0"
+                          lower="-1.69297" upper="${pi}" effort="32.0" vel="3.14"/>
+    <xacro:revolute_joint name="joint6" parent="link5" child="link6"
+                          ax="0" ay="0" az="1" ox="0.076" oy="0.097" oz="0" orx="-1.5708" ory="0" orz="0"
+                          lower="-${2*pi}" upper="${2*pi}" effort="20.0" vel="3.14"/>
 </robot>
