Commit message: Changed camera position

File: nolon_bot_description/urdf/nolon_bot.urdf.xacro (robot description, xacro)
@@ -37,5 +37,5 @@
             <parent link="base_link"/>
             <child link="camera_link"/>
-            <origin xyz="0 0 2" rpy="0 0 0"/>
+            <origin xyz="0.25 0 1.05" rpy="0 0 0"/>
         </joint>
     </xacro:if>

Commit message: Added Moveit

File: nolon_bot_description/urdf/nolon_bot.urdf.xacro (robot description, xacro)
@@ -16,7 +16,7 @@
 -->
 <robot xmlns:xacro="http://www.ros.org/wiki/xacro" name="nolon_bot">
-    <xacro:arg name="use_gazebo" default="true"/>
+    <xacro:arg name="use_gazebo" default="false"/>
     <xacro:property name="use_lidar" value="false"/>
-    <xacro:property name="use_camera" value="true"/>
+    <xacro:property name="use_camera" value="false"/>
     <xacro:include filename="mobile_base/mobile_base.urdf.xacro"/>
     <xacro:include filename="mobile_base/mobile_base.control.xacro"/>

File: nolon_bot_description/urdf/robotic_arm/robotic_arm.control.xacro (robot description, xacro)
@@ -23,5 +23,8 @@
         <!-- Joint 1 Interface -->
         <joint name="joint1">
-            <command_interface name="position"/>
+            <command_interface name="position">
+                <param name="min">${-2.0*pi}</param>
+                <param name="max">${2.0*pi}</param>
+            </command_interface>
             <state_interface name="position"/>
             <state_interface name="velocity"/>
@@ -29,5 +32,8 @@
         <!-- Joint 2 Interface -->
         <joint name="joint2">
-            <command_interface name="position"/>
+            <command_interface name="position">
+                <param name="min">-2.059</param>
+                <param name="max">2.0944</param>
+            </command_interface>
             <state_interface name="position"/>
             <state_interface name="velocity"/>
@@ -35,5 +41,8 @@
         <!-- Joint 3 Interface -->
         <joint name="joint3">
-            <command_interface name="position"/>
+            <command_interface name="position">
+                <param name="min">-3.927</param>
+                <param name="max">0.19198</param>
+            </command_interface>
             <state_interface name="position"/>
             <state_interface name="velocity"/>
@@ -41,5 +50,8 @@
         <!-- Joint 4 Interface -->
         <joint name="joint4">
-            <command_interface name="position"/>
+            <command_interface name="position">
+                <param name="min">${-2.0*pi}</param>
+                <param name="max">${2.0*pi}</param>
+            </command_interface>
             <state_interface name="position"/>
             <state_interface name="velocity"/>
@@ -47,5 +59,8 @@
         <!-- Joint 5 Interface -->
         <joint name="joint5">
-            <command_interface name="position"/>
+            <command_interface name="position">
+                <param name="min">-1.69297</param>
+                <param name="max">${pi}</param>
+            </command_interface>
             <state_interface name="position"/>
             <state_interface name="velocity"/>
@@ -53,5 +68,8 @@
         <!-- Joint 6 Interface -->
         <joint name="joint6">
-            <command_interface name="position"/>
+            <command_interface name="position">
+                <param name="min">${-2.0*pi}</param>
+                <param name="max">${2.0*pi}</param>
+            </command_interface>
             <state_interface name="position"/>
             <state_interface name="velocity"/>

File: nolon_bot_description/urdf/robotic_arm/robotic_arm.urdf.xacro (robot description, xacro)
@@ -18,4 +18,5 @@
 -->
 <robot xmlns:xacro="http://www.ros.org/wiki/xacro" name="robotic_arm">
+    <xacro:arg name="use_gazebo" default="false"/>
     <!-- ================= CHECK USAGE ================= -->
     <!-- Conditional mesh path -->
