Commit message: Added RGBD camera

File: nolon_bot_description/urdf/containment/containment_box.urdf.xacro (robot description, xacro)
@@ -17,11 +17,10 @@
 <robot xmlns:xacro="http://www.ros.org/wiki/xacro" name="mobile_base">
   <!-- ================= CHECK USAGE ================= -->
-  <xacro:arg name="use_gazebo" default="true"/>
   <!-- Conditional mesh path -->
   <xacro:if value="$(arg use_gazebo)">
-    <xacro:property name="mesh_path" value="file:///home/aayush/Internship/nolon_bot_ws/src/nolon_bot_description/meshes/containment/"/>
+    <xacro:property name="mesh_path" value="$(find nolon_bot_description)/meshes/containment/"/>
   </xacro:if>
   <xacro:unless value="$(arg use_gazebo)">
-    <xacro:property name="mesh_path" value="$(find nolon_bot_description)/meshes/"/>
+    <xacro:property name="mesh_path" value="file:///home/aayush/Internship/nolon_bot_ws/src/nolon_bot_description/meshes/containment/"/>
   </xacro:unless>
   <!-- ================= MACROS ================= -->

File: nolon_bot_description/urdf/mobile_base/mobile_base.urdf.xacro (robot description, xacro)
@@ -19,8 +19,8 @@
   <!-- Conditional mesh path -->
   <xacro:if value="$(arg use_gazebo)">
-    <xacro:property name="mesh_path" value="file:///home/aayush/Internship/nolon_bot_ws/src/nolon_bot_description/meshes/mobile_base/"/>
+    <xacro:property name="mesh_path" value="$(find nolon_bot_description)/meshes/mobile_base/"/>
   </xacro:if>
   <xacro:unless value="$(arg use_gazebo)">
-    <xacro:property name="mesh_path" value="$(find nolon_bot_description)/meshes/"/>
+    <xacro:property name="mesh_path" value="file:///home/aayush/Internship/nolon_bot_ws/src/nolon_bot_description/meshes/mobile_base/"/>
   </xacro:unless>
   <!-- ================= MACROS ================= -->

File: nolon_bot_description/urdf/nolon_bot.urdf.xacro (robot description, xacro)
@@ -16,5 +16,7 @@
 -->
 <robot xmlns:xacro="http://www.ros.org/wiki/xacro" name="nolon_bot">
+    <xacro:arg name="use_gazebo" default="true"/>
     <xacro:property name="use_lidar" value="false"/>
+    <xacro:property name="use_camera" value="true"/>
     <xacro:include filename="mobile_base/mobile_base.urdf.xacro"/>
     <xacro:include filename="mobile_base/mobile_base.control.xacro"/>
@@ -30,5 +32,12 @@
         </joint>
     </xacro:if>
-<!-- -0.1 0 0.5-->
+    <xacro:if value="${use_camera}">
+        <xacro:include filename="sensors/camera.sensor.xacro"/>
+        <joint name="camera_joint" type="fixed">
+            <parent link="base_link"/>
+            <child link="camera_link"/>
+            <origin xyz="0 0 2" rpy="0 0 0"/>
+        </joint>
+    </xacro:if>
     <joint name="containment_to_mobile_base" type="fixed">
         <parent link="base_link"/>
@@ -36,5 +45,4 @@
         <origin xyz="0 0 0" rpy="0 0 0"/>
     </joint>
-    <!-- <link name="world"/> -->
     <joint name="robotic_arm_to_containment" type="fixed">
         <parent link="containment_box"/>
@@ -47,4 +55,7 @@
             <controller_manager_node_name>controller_manager</controller_manager_node_name>
         </plugin>
+        <plugin filename="gz-sim-sensors-system" name="gz::sim::systems::Sensors">
+            <render_engine>ogre2</render_engine>
+        </plugin>
     </gazebo>
 </robot>

File: nolon_bot_description/urdf/robotic_arm/robotic_arm.urdf.xacro (robot description, xacro)
@@ -19,11 +19,10 @@
 <robot xmlns:xacro="http://www.ros.org/wiki/xacro" name="robotic_arm">
     <!-- ================= CHECK USAGE ================= -->
-    <xacro:arg name="use_gazebo" default="true"/>
     <!-- Conditional mesh path -->
     <xacro:if value="$(arg use_gazebo)">
-        <xacro:property name="mesh_path" value="file:///home/aayush/Internship/nolon_bot_ws/src/nolon_bot_description/meshes/robotic_arm/"/>
+        <xacro:property name="mesh_path" value="$(find nolon_bot_description)/meshes/robotic_arm/"/>
     </xacro:if>
     <xacro:unless value="$(arg use_gazebo)">
-        <xacro:property name="mesh_path" value="$(find nolon_bot_description)/meshes/robotic_arm/"/>
+        <xacro:property name="mesh_path" value="file:///home/aayush/Internship/nolon_bot_ws/src/nolon_bot_description/meshes/robotic_arm/"/>
     </xacro:unless>
     <!-- ================= MATERIALS ================= -->

File: nolon_bot_description/urdf/sensors/lidar.sensor.xacro (robot description, xacro)
@@ -43,9 +43,4 @@
         </collision>
     </link>
-    <gazebo>
-        <plugin filename="gz-sim-sensors-system" name="gz::sim::systems::Sensors">
-            <render_engine>ogre2</render_engine>
-        </plugin>
-    </gazebo>
     <gazebo reference="lidar_link">
         <sensor name="lidar_link" type="gpu_lidar">

Commit message: Added usd file for isaac sim

File: nolon_bot_description/urdf/containment/containment_box.urdf.xacro (robot description, xacro)
@@ -26,40 +26,50 @@
   <!-- ================= MACROS ================= -->
   <!-- Generic mesh link -->
-<xacro:macro name="mesh_link" params="name mesh mass ixx iyy izz ixy ixz iyz ox oy oz orx ory orz">
-  <link name="${name}">
-    <visual>
+  <xacro:macro name="mesh_link" params="name mesh mass ixx iyy izz ixy ixz iyz ox oy oz orx ory orz">
+    <link name="${name}">
+      <visual>
+        <origin xyz="${ox} ${oy} ${oz}" rpy="${orx} ${ory} ${orz}"/>
+        <geometry>
+          <mesh filename="${mesh_path}${mesh}"/>
+        </geometry>
+        <material name="DarkGreyShiny">
+          <!-- Darker grey -->
+          <color rgba="0.3 0.3 0.3 1"/>
+        </material>
+      </visual>
+      <collision>
+        <origin xyz="${ox} ${oy} ${oz}" rpy="${orx} ${ory} ${orz}"/>
+        <geometry>
+          <mesh filename="${mesh_path}${mesh}"/>
+        </geometry>
+      </collision>
+      <inertial>
+        <mass value="${mass}"/>
+        <origin xyz="${ox} ${oy} ${oz}" rpy="${orx} ${ory} ${orz}"/>
+        <inertia ixx="${ixx}" iyy="${iyy}" izz="${izz}" ixy="${ixy}" ixz="${ixz}" iyz="${iyz}"/>
+      </inertial>
+    </link>
+    <gazebo reference="${name}">
+      <material>Gazebo/Grey</material>
+      <material>
+        <ambient>0.3 0.3 0.3 1</ambient>
+        <diffuse>0.3 0.3 0.3 1</diffuse>
+        <specular>0.6 0.6 0.6 1</specular>
+        <emissive>0 0 0 1</emissive>
+      </material>
+    </gazebo>
+  </xacro:macro>
+  <xacro:macro name="fixed_joint" params="parent child ox oy oz orx ory orz">
+    <joint name="${parent}_to_${child}" type="fixed">
+      <parent link="${parent}"/>
+      <child link="${child}"/>
       <origin xyz="${ox} ${oy} ${oz}" rpy="${orx} ${ory} ${orz}"/>
-      <geometry>
-        <mesh filename="${mesh_path}${mesh}"/>
-      </geometry>
-      <material name="DarkGreyShiny">
-        <!-- Darker grey -->
-        <color rgba="0.3 0.3 0.3 1"/>
-      </material>
-    </visual>
-    <collision>
-      <origin xyz="${ox} ${oy} ${oz}" rpy="${orx} ${ory} ${orz}"/>
-      <geometry>
-        <mesh filename="${mesh_path}${mesh}"/>
-      </geometry>
-    </collision>
-    <inertial>
-      <mass value="${mass}"/>
-      <origin xyz="${ox} ${oy} ${oz}" rpy="${orx} ${ory} ${orz}"/>
-      <inertia ixx="${ixx}" iyy="${iyy}" izz="${izz}" ixy="${ixy}" ixz="${ixz}" iyz="${iyz}"/>
-    </inertial>
-  </link>
-  <gazebo reference="${name}">
-    <material>Gazebo/Grey</material>
-    <material>
-      <ambient>0.3 0.3 0.3 1</ambient>
-      <diffuse>0.3 0.3 0.3 1</diffuse>
-      <specular>0.6 0.6 0.6 1</specular>
-      <emissive>0 0 0 1</emissive>
-    </material>
-  </gazebo>
-</xacro:macro>
+    </joint>
+  </xacro:macro>
   <!-- ================= ROBOT STRUCTURE ================= -->
   <!-- Containment Box -->
-  <xacro:mesh_link name="containment_box" mesh="containment_box.stl" mass="5.0" ixx="2.0" iyy="2.0" izz="2.0" ixy="0" ixz="0" iyz="0" ox="0" oy="0" oz="0" orx="0" ory="0" orz="0"/>
+  <xacro:mesh_link name="containment_box" mesh="containment_box_0.stl" mass="5.0" ixx="2.0" iyy="2.0" izz="2.0" ixy="0" ixz="0" iyz="0" ox="0" oy="0" oz="0" orx="0" ory="0" orz="0"/>
+  <!-- Text Box -->
+  <!-- <xacro:mesh_link name="text" mesh="text.stl" mass="0.01" ixx="0.001" iyy="0.001" izz="0.001" ixy="0" ixz="0" iyz="0" ox="0" oy="0" oz="0" orx="0" ory="0" orz="0"/>
+  <xacro:fixed_joint parent="containment_box" child="text"  ox="0" oy="0" oz="0" orx="0" ory="0" orz="0"/> -->
 </robot>
